Commit message: slam with navigation

File: model/Lidar.xacro (robot description, xacro)
@@ -4,5 +4,5 @@
         <parent link = "chassis"/>
         <child link = "laser_frame"/>
-        <origin xyz = " 0.1 0 0.175" rpy = "0 0 0"/>
+        <origin xyz = " 0.1 0 0.0" rpy = "0 0 0"/>
     </joint>
     <link name = "laser_frame">
@@ -24,5 +24,5 @@
     <gazebo reference = "laser_frame">
         <material>Gazebo/Red</material>
-        <sensor name = "lase" type = "ray">
+        <sensor name = "laser" type = "ray">
             <pose> 0 0 0 0 0 0</pose>
             <visualize> true</visualize>

File: model/robot_core.xacro (robot description, xacro)
@@ -19,4 +19,12 @@
     <!-- Base link -->
     <link name="base_link">
+    </link>
+    <!-- Base footprint -->
+    <joint name="base_footprint_joint" type="fixed">
+        <parent link="base_link" />
+        <child link="base_footprint" />
+        <origin xyz="0 0 0" rpy="0 0 0"/>
+    </joint>
+    <link name="base_footprint">
     </link>
     <!-- Chassis link -->
@@ -93,5 +101,5 @@
         <parent link="chassis"/>
         <child link="caster_wheel"/>
-        <origin xyz="0.24 0 0"/>
+        <origin xyz="0.3 0 0"/>
     </joint>
     <link name="caster_wheel">
@@ -107,5 +115,5 @@
             </geometry>
         </collision>
-        <xacro:inertial_sphere mass="0.5" radius="0.05">
+        <xacro:inertial_sphere mass="4" radius="0.05">
             <origin xyz="0 0 0" rpy="0 0 0"/>
         </xacro:inertial_sphere>

Commit message: tuning and substituting some nav algorithms + robot shape + cost map parameters for smarter motion

File: model/Lidar.xacro (robot description, xacro)
@@ -4,5 +4,7 @@
         <parent link = "chassis"/>
         <child link = "laser_frame"/>
-        <origin xyz = " 0.1 0 0.0" rpy = "0 0 0"/>
+        <origin xyz = "0.15 0 0.08" rpy = "0 0 0"/>
+        <!-- <axis xyz="1 0 0"> -->
+        <!-- <limit lower="-1.57" upper="1.57" effort="1.0" velocity="1.0"> -->
     </joint>
     <link name = "laser_frame">
@@ -38,5 +40,5 @@
                 </scan>
                 <range>
-                    <min>0.3</min>
+                    <min>0.22</min>
                     <max>12</max>
                     <resolution>0.01</resolution>

File: model/robot_core.xacro (robot description, xacro)
@@ -36,7 +36,7 @@
     <link name="chassis">
         <visual>
-            <origin xyz="0.15 0 0.075" />
+            <origin xyz="0.15 0 0.05" />
             <geometry>
-                <box size="0.3 0.3 0.15" />
+                <box size="0.3 0.3 0.05" />
             </geometry>
             <material name="white" />
@@ -45,8 +45,8 @@
             <origin xyz="0.15 0 0.075" />
             <geometry>
-                <box size="0.3 0.3 0.15" />
+                <box size="0.3 0.3 0.05" />
             </geometry>
         </collision>
-        <xacro:inertial_box mass="1" x="0.3" y="0.3" z="0.15">
+        <xacro:inertial_box mass="1" x="0.3" y="0.3" z="0.05">
             <origin xyz="0.15 0 0.075" rpy="0 0 0"/>
         </xacro:inertial_box>

Commit message: final robot control

File: model/Lidar.xacro (robot description, xacro)
@@ -11,5 +11,5 @@
         <visual>
             <geometry>
-                <cylinder radius="0.05" length="0.04" />
+                <cylinder radius="0.05" length="0.02" />
             </geometry>
             <material name="blue" />
@@ -17,8 +17,8 @@
         <collision>
             <geometry>
-                <cylinder radius="0.05" length="0.04" />
+                <cylinder radius="0.05" length="0.02" />
             </geometry>
         </collision>
-        <xacro:inertial_cylinder mass="1" length="0.04" radius="0.05">
+        <xacro:inertial_cylinder mass="1" length="0.02" radius="0.05">
             <origin xyz="0 0 0" rpy="0 0 0"/>
         </xacro:inertial_cylinder>
